Commit message: Add OnRobot 2FG7 module STL file for iiwa7_R robot, left finger as EE

File: jrl/urdfs/iiwa7_L/iiwa7_L_updated.urdf (robot description, URDF)
Before this commit: robot iiwa7_0, 14 links, 13 joints
Joints:
- joint lbr1_world_iiwa_joint: origin xyz=0.3682   -0.1842    0.7014 rpy=0.0039    -0.0030   -0.0161 -> xyz=0.3682 -0.1842 0.7014 rpy=0.0039 -0.0030 -0.0161

Commit message: Update visualization script to load updated robot URDF and improve path resolution
- Changed the URDF file loaded for the robot from "dual_iiwa7" to "iiwa7_R_updated".
- Added a line to change the working directory to ensure mesh paths are resolved correctly.
- Included print statements to confirm successful loading of the robot and display the number of joints.
- Suggested updating Klampt to resolve potential issues with the Qt backend.

File: jrl/urdfs/iiwa7_L/iiwa7_L_updated.urdf (robot description, URDF)
Before this commit: robot iiwa7_0, 14 links, 13 joints
Links:
- link lbr1_left_finger_link: geometry collision mesh filename=urdfs/iiwa7_L/meshes/onrobot_2fg7/2fg7_gripper_left.stl; visual mesh filename=urdfs/iiwa7_L/meshes/onrobot_2fg7/2fg7_gripper_left.stl
- link lbr1_link_gripper: geometry collision cylinder length=0.12 radius=0.055; visual mesh filename=urdfs/iiwa7_L/meshes/onrobot_2fg7/2fg7_module.stl
- link lbr1_right_finger_link: geometry collision mesh filename=urdfs/iiwa7_L/meshes/onrobot_2fg7/2fg7_gripper_right.stl; visual mesh filename=urdfs/iiwa7_L/meshes/onrobot_2fg7/2fg7_gripper_right.stl

File: jrl/urdfs/iiwa7_R/iiwa7_R_updated.urdf (robot description, URDF)
Before this commit: robot iiwa7_0, 14 links, 13 joints
Links:
- link lbr2_left_finger_link: geometry collision mesh filename=urdfs/iiwa7_R/meshes/onrobot_2fg7/2fg7_gripper_left.stl; visual mesh filename=urdfs/iiwa7_R/meshes/onrobot_2fg7/2fg7_gripper_left.stl
- link lbr2_link_gripper: geometry collision cylinder length=0.12 radius=0.055; visual mesh filename=urdfs/iiwa7_R/meshes/onrobot_2fg7/2fg7_module.stl
- link lbr2_right_finger_link: geometry collision mesh filename=urdfs/iiwa7_R/meshes/onrobot_2fg7/2fg7_gripper_right.stl; visual mesh filename=urdfs/iiwa7_R/meshes/onrobot_2fg7/2fg7_gripper_right.stl

Commit message: Update URDF and visualization scripts for IIWA7_L robot integration and improve forward kinematics handling

File: jrl/urdfs/iiwa7_L/iiwa7_L_updated.urdf (robot description, URDF)
Before this commit: robot iiwa7_0, 14 links, 13 joints
Links:
- link lbr1_link_gripper: geometry collision mesh filename=urdfs/iiwa7_R/meshes/onrobot_2fg7/2fg7_module.stl; visual mesh filename=urdfs/iiwa7_L/meshes/onrobot_2fg7/2fg7_module.stl
Joints:
- joint lbr1_joint_gripper: origin xyz=0 0 0 rpy=0 0 0 -> xyz=0 0 0 rpy=1.5708 0 1.5708
- joint lbr1_left_finger_joint: origin xyz=0 -0.006 0 rpy=0 0 0 -> xyz=0 0 0 rpy=0 0 0
- joint lbr1_right_finger_joint: origin xyz=0 0.006 0 rpy=0 0 0 -> xyz=0 0 0 rpy=0 0 0

Commit message: Refactor collision pairs and update end effector links for IIWA7_L and IIWA7_R robots; add true end effector links in URDF files.

File: jrl/urdfs/iiwa7_L/iiwa7_L_updated.urdf (robot description, URDF)
Before this commit: robot iiwa7_0, 14 links, 13 joints
Links:
- added link lbr1_true_ee_link
Joints:
- added joint lbr1_true_ee_joint: type fixed, parent lbr1_left_finger_link, child lbr1_true_ee_link, origin xyz=0 0.14 0 rpy=0 0 0

File: jrl/urdfs/iiwa7_R/iiwa7_R_updated.urdf (robot description, URDF)
Before this commit: robot iiwa7_0, 14 links, 13 joints
Links:
- added link lbr2_true_ee_link
Joints:
- added joint lbr2_true_ee_joint: type fixed, parent lbr2_left_finger_link, child lbr2_true_ee_link, origin xyz=0 0.14 0 rpy=0 0 0

Commit message: Refactor code structure for improved readability and maintainability

File: jrl/urdfs/iiwa7_L/iiwa7_L_updated.urdf (robot description, URDF)
Before this commit: robot iiwa7_0, 15 links, 14 joints
Links:
- removed link lbr1_gripper_link_ee
- removed link lbr1_link_ee
- link lbr1_link_gripper: geometry collision mesh filename=urdfs/iiwa7_L/meshes/collision/lbr1_gripper_blender.stl; visual mesh filename=urdfs/iiwa7_L/meshes/collision/lbr1_gripper_blender.stl
- link lbr1_true_ee_link: mass None -> 0.001; geometry collision mesh filename=urdfs/iiwa7_L/meshes/collision/small_ball.stl; visual mesh filename=urdfs/iiwa7_L/meshes/collision/small_ball.stl
Joints:
- removed joint lbr1_gripper_ee
- removed joint lbr1_joint_gripper
- joint lbr1_joint_ee: child lbr1_link_ee -> lbr1_link_gripper; origin xyz=0.0 0.0 0.045 rpy=0.0 0.0 0.0 -> xyz=0.0 0.0 0.105 rpy=0.0 0.0 0.0
- joint lbr1_left_finger_joint: origin xyz=0 0 0 rpy=0 0 0 -> xyz=0.012 0 0.061 rpy=0 0 0
- joint lbr1_right_finger_joint: origin xyz=0 0 0 rpy=0 0 0 -> xyz=-0.012 0 0.061 rpy=0 0 0
- joint lbr1_true_ee_joint: origin xyz=0 0.14 0 rpy=0 0 0 -> xyz=-0.012 0 0.03 rpy=0 0 0
