Commit message: Update IIWA7 URDF and capsule configurations for improved collision handling and visualization

File: jrl/urdfs/iiwa7_R/iiwa7_R_updated.urdf (robot description, URDF)
Before this commit: robot iiwa7_0, 14 links, 13 joints
Links:
- link lbr2_link_ee: geometry visual sphere radius=0.001
- link lbr2_link_gripper: geometry collision mesh filename=urdfs/iiwa7_R/meshes/onrobot_2fg7/2fg7_module.stl; visual mesh filename=urdfs/iiwa7_R/meshes/onrobot_2fg7/2fg7_module.stl
Joints:
- joint lbr2_joint_gripper: origin xyz=0 0 0 rpy=0 0 0 -> xyz=0 0 0 rpy=1.5708 0 1.5708
- joint lbr2_left_finger_joint: origin xyz=0 -0.006 0 rpy=0 0 0 -> xyz=0 0 0 rpy=0 0 0
- joint lbr2_right_finger_joint: origin xyz=0 0.006 0 rpy=0 0 0 -> xyz=0 0 0 rpy=0 0 0

Commit message: Refactor code structure for improved readability and maintainability

File: jrl/urdfs/iiwa7_R/iiwa7_R_updated.urdf (robot description, URDF)
Before this commit: robot iiwa7_0, 15 links, 14 joints
Links:
- removed link lbr2_gripper_link_ee
- removed link lbr2_link_ee
- link lbr2_link_gripper: geometry collision mesh filename=urdfs/iiwa7_R/meshes/collision/lbr2_gripper_blender.stl; visual mesh filename=urdfs/iiwa7_R/meshes/collision/lbr2_gripper_blender.stl
- link lbr2_true_ee_link: mass None -> 0.001; geometry collision mesh filename=urdfs/iiwa7_R/meshes/collision/small_ball.stl; visual mesh filename=urdfs/iiwa7_R/meshes/collision/small_ball.stl
Joints:
- removed joint lbr2_gripper_ee
- removed joint lbr2_joint_gripper
- joint lbr2_joint_ee: child lbr2_link_ee -> lbr2_link_gripper; origin xyz=0.0 0.0 0.045 rpy=0.0 0.0 0.0 -> xyz=0.0 0.0 0.105 rpy=0.0 0.0 0.0
- joint lbr2_left_finger_joint: origin xyz=0 0 0 rpy=0 0 0 -> xyz=0.012 0 0.061 rpy=0 0 0
- joint lbr2_right_finger_joint: origin xyz=0 0 0 rpy=0 0 0 -> xyz=-0.012 0 0.061 rpy=0 0 0
- joint lbr2_true_ee_joint: origin xyz=0 0.14 0 rpy=0 0 0 -> xyz=-0.012 0 0.03 rpy=0 0 0
